File: blogic.sch (KiCad schematic (older format))
At the start: 21 parts

Commit message: wip
Parts:
- added D1: LED, ~, symbol LED
- added P1, P2: CONN_9, symbol CONN_9
- added R1: 330R, ~, symbol R
- added R10, R11, R12, R13, R14, R15, R16, R17, R18, R19, R20, R21, R6, R7, R8, R9: 51R, ~, symbol R
- gave numbers to parts that had none: 21
Connections:
- net GND: now also P1.1 (P1), P2.1 (P1), R1.2
- net VCC: now also D1.1 (A)
- net at DD1.1 (FD13): now also R19.1
- net at DD1.2 (FD14): now also R20.1
- net at DD1.25 (FD0): now also R6.1
- net at DD1.26 (FD1): now also R7.1
- net at DD1.27 (FD2): now also R8.1
- net at DD1.28 (FD3): now also R9.1
- net at DD1.29 (FD4): now also R10.1
- net at DD1.3 (FD15): now also R21.1
- net at DD1.30 (FD5): now also R11.1
- net at DD1.31 (FD6): now also R12.1
- net at DD1.32 (FD7): now also R13.1
- net at DD1.52 (FD8): now also R14.1
- net at DD1.53 (FD9): now also R15.1
- net at DD1.54 (FD10): now also R16.1
- net at DD1.55 (FD11): now also R17.1
- net at DD1.56 (FD12): now also R18.1
- new net: P1.2 (P2), R6.2
- new net: P1.3 (P3), R7.2
- new net: P1.4 (P4), R8.2
- new net: P1.5 (P5), R9.2
- new net: P1.6 (P6), R10.2
- new net: P1.7 (P7), R11.2
- new net: P1.8 (P8), R12.2
- new net: P1.9 (P9), R13.2
- new net: P2.2 (P2), R14.2
- new net: P2.3 (P3), R15.2
- new net: P2.4 (P4), R16.2
- new net: P2.5 (P5), R17.2
- new net: P2.6 (P6), R18.2
- new net: P2.7 (P7), R19.2
- new net: P2.8 (P8), R20.2
- new net: P2.9 (P9), R21.2
- new net: D1.2 (K), R1.1
Other:
- moved on the sheet: C1, C10, C11, C2, C3, C4, C5, C6, C7, C8, C9, CON1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
