File: blogic.kicad_pcb (KiCad board)
At the start: 2 copper layers, 50 x 50 mm, 46 parts, among them CON1 USB-MINI-B, P1 CONN_9, P2 CONN_9, U1 24C16, U2 AMS1117_3V3, X1 24M

Commit message: pcb
Routing:
- net (no net): track 0.00 -> 1.07 mm, vias 0 -> 1
Changed lines of the file:
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@@
     (thickness 1.6)
     (drawings 7)
-    (tracks 436)
+    (tracks 439)
     (zones 0)
     (modules 46)
@@
   )
   (layers
-    (15 F.Cu signal hide)
+    (15 F.Cu signal)
     (0 B.Cu signal)
     (16 B.Adhes user)
-    (17 F.Adhes user hide)
+    (17 F.Adhes user)
     (18 B.Paste user)
-    (19 F.Paste user hide)
+    (19 F.Paste user)
     (20 B.SilkS user)
-    (21 F.SilkS user hide)
+    (21 F.SilkS user)
     (22 B.Mask user)
-    (23 F.Mask user hide)
+    (23 F.Mask user)
     (24 Dwgs.User user)
     (25 Cmts.User user)
@@
     (mod_text_size 1 1)
     (mod_text_width 0.15)
-    (pad_size 3.8 1.92)
-    (pad_drill 0)
+    (pad_size 0.89916 0.89916)
+    (pad_drill 0.89916)
     (pad_to_mask_clearance 0)
     (aux_axis_origin 0 0)
-    (visible_elements FFFFDF3F)
+    (visible_elements FFFFFF3F)
     (pcbplotparams
-      (layerselection 3178497)
+      (layerselection 15761409)
       (usegerberextensions true)
-      (excludeedgelayer true)
+      (excludeedgelayer false)
       (linewidth 152400)
       (plotframeref false)
@@
       (psa4output false)
       (plotreference true)
-      (plotvalue true)
+      (plotvalue false)
       (plotothertext true)
       (plotinvisibletext false)
@@
       (outputformat 1)
       (mirror false)
-      (drillshape 1)
+      (drillshape 0)
       (scaleselection 1)
-      (outputdirectory ""))
+      (outputdirectory ./gerber/))
   )
   (net 0 "")
@@
       (net 4 GND)
     )
-    (pad "" np_thru_hole circle (at 0.8509 -2.19964) (size 0.89916 0.89916) (drill 0.89916)
+    (pad "" thru_hole circle (at 0.8509 -2.19964) (size 0.89916 0.89916) (drill 0.89916)
       (layers *.Cu *.Mask F.SilkS)
     )
-    (pad 2 np_thru_hole circle (at 0.8509 2.19964) (size 0.89916 0.89916) (drill 0.89916)
+    (pad 2 thru_hole circle (at 0.8509 2.19964) (size 0.89916 0.89916) (drill 0.89916)
       (layers *.Cu *.Mask F.SilkS)
       (net 18 N-0000024)
+    )
+    (model usb_B_mini_smd.wrl
+      (at (xyz -0.01 0 0))
+      (scale (xyz 1 1 1))
+      (rotate (xyz 0 0 90))
     )
   )
@@
       (layers F.Cu F.Paste F.Mask)
       (net 43 N-000008)
+    )
+    (model smd/vsop56.wrl
+      (at (xyz 0 0 0))
+      (scale (xyz 0.25 0.25 0.75))
+      (rotate (xyz 0 0 0))
     )
   )
@@
       (layers F.Cu F.Paste F.Mask)
       (net 24 N-0000030)
+    )
+    (model pin_strip_9x2.wrl
+      (at (xyz -0.1 0 -0.03))
+      (scale (xyz 1 1 1))
+      (rotate (xyz 90 0 270))
     )
   )
@@
   (gr_line (start 215 175) (end 215 125) (angle 90) (layer Edge.Cuts) (width 0.15))
   (gr_line (start 165 175) (end 215 175) (angle 90) (layer Edge.Cuts) (width 0.15))
+  (segment (start 183.515 153.289) (end 183.515 152.654) (width 0.254) (layer F.Cu) (net 0))
+  (segment (start 183.642 152.527) (end 183.642 152.273) (width 0.254) (layer B.Cu) (net 0))
+  (via (at 183.642 152.527) (size 0.889) (layers F.Cu B.Cu) (net 0))
+  (segment (start 183.515 152.654) (end 183.642 152.527) (width 0.254) (layer F.Cu) (net 0))
   (segment (start 176.403 141.986) (end 176.149 142.24) (width 0.508) (layer F.Cu) (net 1))
   (segment (start 176.149 142.24) (end 174.1805 142.24) (width 0.508) (layer F.Cu) (net 1))
@@
   (segment (start 194.056 161.798) (end 193.04 161.798) (width 0.254) (layer F.Cu) (net 3))
   (segment (start 195.3975 160.4565) (end 194.056 161.798) (width 0.254) (layer F.Cu) (net 3))
-  (segment (start 212.344 160.16) (end 212.344 162.306) (width 0.254) (layer B.Cu) (net 4) (status 400000))
+  (segment (start 212.344 160.16) (end 212.344 162.306) (width 0.254) (layer B.Cu) (net 4))
   (segment (start 212.344 162.306) (end 212.344 162.052) (width 0.254) (layer F.Cu) (net 4))
   (via (at 212.344 162.306) (size 0.889) (layers F.Cu B.Cu) (net 4))
-  (segment (start 212.344 160.16) (end 209.436 160.16) (width 0.254) (layer F.Cu) (net 4) (status 400000))
+  (segment (start 212.344 160.16) (end 209.436 160.16) (width 0.254) (layer F.Cu) (net 4))
   (via (at 209.296 160.02) (size 0.889) (layers F.Cu B.Cu) (net 4))
   (segment (start 209.436 160.16) (end 209.296 160.02) (width 0.254) (layer F.Cu) (net 4))
@@
   (segment (start 198.5725 153.2175) (end 198.5725 154.7625) (width 0.254) (layer F.Cu) (net 13))
   (segment (start 201.93 149.86) (end 198.5725 153.2175) (width 0.254) (layer F.Cu) (net 13))
-  (segment (start 184.15 152.146) (end 183.642 152.146) (width 0.254) (layer F.Cu) (net 14))
-  (segment (start 184.15 152.146) (end 189.23 152.146) (width 0.254) (layer F.Cu) (net 14))
+  (segment (start 184.404 152.146) (end 189.23 152.146) (width 0.254) (layer F.Cu) (net 14))
   (segment (start 189.23 152.146) (end 190.3175 153.2335) (width 0.254) (layer F.Cu) (net 14))
   (segment (start 190.3175 154.7625) (end 190.3175 153.2335) (width 0.254) (layer F.Cu) (net 14))
   (segment (start 180.848 150.622) (end 180.226 150) (width 0.254) (layer F.Cu) (net 14))
-  (segment (start 182.118 150.622) (end 180.848 150.622) (width 0.254) (layer F.Cu) (net 14))
-  (segment (start 183.642 152.146) (end 182.118 150.622) (width 0.254) (layer F.Cu) (net 14))
+  (segment (start 183.007 150.622) (end 180.848 150.622) (width 0.254) (layer F.Cu) (net 14))
+  (segment (start 184.531 152.146) (end 183.007 150.622) (width 0.254) (layer F.Cu) (net 14))
   (segment (start 172.54732 150) (end 180.226 150) (width 0.254) (layer F.Cu) (net 14))
   (segment (start 203.5175 157.48) (end 201.93 157.48) (width 0.254) (layer F.Cu) (net 15))
@@
   (segment (start 190.9525 152.9795) (end 190.9525 154.7625) (width 0.254) (layer F.Cu) (net 18))
   (segment (start 189.484 151.511) (end 190.9525 152.9795) (width 0.254) (layer F.Cu) (net 18))
-  (segment (start 183.769002 151.511) (end 189.484 151.511) (width 0.254) (layer F.Cu) (net 18))
-  (segment (start 182.245002 149.987) (end 183.769002 151.511) (width 0.254) (layer F.Cu) (net 18))
-  (segment (start 181.102 149.987) (end 182.245002 149.987) (width 0.254) (layer F.Cu) (net 18))
+  (segment (start 184.912002 151.511) (end 189.484 151.511) (width 0.254) (layer F.Cu) (net 18))
+  (segment (start 183.388002 149.987) (end 184.912002 151.511) (width 0.254) (layer F.Cu) (net 18))
+  (segment (start 181.102 149.987) (end 183.388002 149.987) (width 0.254) (layer F.Cu) (net 18))
   (segment (start 180.4419 149.3269) (end 181.102 149.987) (width 0.254) (layer F.Cu) (net 18))
   (segment (start 180.4419 149.1999) (end 180.4419 149.3269) (width 0.254) (layer F.Cu) (net 18))
@@
   (segment (start 202.03 165) (end 199.7075 167.3225) (width 0.254) (layer F.Cu) (net 45))
   (segment (start 179.07 146.685) (end 179.07 148.717) (width 0.508) (layer B.Cu) (net 45))
-  (segment (start 184.531 153.035) (end 185.42 153.035) (width 0.508) (layer B.Cu) (net 45))
-  (segment (start 181.483 156.083) (end 184.531 153.035) (width 0.508) (layer B.Cu) (net 45))
-  (segment (start 178.054 156.083) (end 181.483 156.083) (width 0.508) (layer B.Cu) (net 45))
+  (segment (start 184.785 153.035) (end 185.42 153.035) (width 0.508) (layer B.Cu) (net 45))
+  (segment (start 181.737 156.083) (end 184.785 153.035) (width 0.508) (layer B.Cu) (net 45))
+  (segment (start 178.054 156.083) (end 181.737 156.083) (width 0.508) (layer B.Cu) (net 45))
   (segment (start 177.038 155.194) (end 178.054 156.083) (width 0.508) (layer B.Cu) (net 45))
   (segment (start 177.038 150.749) (end 177.038 155.194) (width 0.508) (layer B.Cu) (net 45))
